File: kicad/boardloaf-he.kicad_pcb (KiCad board)
At the start: 2 copper layers, 100 x 100 mm, 49 parts, among them J1 AudioJack4, J2 AudioJack4, SW1 SW_Push, SW10 SW_Push, SW11 SW_Push, SW12 SW_Push, SW13 SW_Push, SW14 SW_Push, SW15 SW_Push, SW16 SW_Push, SW17 SW_Push, SW18 SW_Push, SW2 SW_Push, SW3 SW_Push, SW4 SW_Push, SW5 SW_Push, SW6 SW_Push, SW7 SW_Push, SW8 SW_Push, SW9 SW_Push, U1 74HC4051, U2 74HC4051, U3 74HC4051

Commit message: Made schematic sync with PCB
Parts:
- C1, C10, C11, C12, C13, C14, C15, C16, C17, C18, C19, C2, C20, C21, C3, C4, C5, C6, C7, C8, C9: value 0805 -> 1uF
- SW1, SW10, SW11, SW12, SW13, SW14, SW15, SW16, SW17, SW18, SW2, SW3, SW4, SW5, SW6, SW7, SW8, SW9: value SW_Push -> SLSS49E
- turned C19 to -90 degrees
- turned C20 to -90 degrees
- turned C21 to -90 degrees
- renumbered MCU to MCU1
Connections:
- C19 pad 1: GND -> VCC
- C19 pad 2: VCC -> GND
- C20 pad 1: GND -> VCC
- C20 pad 2: VCC -> GND
- C21 pad 1: GND -> VCC
- C21 pad 2: VCC -> GND
- MCU1 pad 0: (no net) -> unconnected-(MCU1-Pad0)
- MCU1 pad 1: (no net) -> unconnected-(MCU1-Pad1)
- MCU1 pad 10: (no net) -> unconnected-(MCU1-Pad10)
- MCU1 pad 11: (no net) -> unconnected-(MCU1-Pad11)
- MCU1 pad 12: (no net) -> unconnected-(MCU1-Pad12)
- MCU1 pad 13: (no net) -> unconnected-(MCU1-Pad13)
- MCU1 pad 2: (no net) -> unconnected-(MCU1-Pad2)
- MCU1 pad 29: X -> unconnected-(MCU1-Pad29)
- MCU1 pad 3: (no net) -> unconnected-(MCU1-Pad3)
- MCU1 pad 4: (no net) -> unconnected-(MCU1-Pad4)
- MCU1 pad 5: (no net) -> unconnected-(MCU1-Pad5)
- MCU1 pad 9: (no net) -> unconnected-(MCU1-Pad9)

Commit message: Rev 1.1 draft. Mux on both sides
Parts:
- removed the JP1 at (99.3, 89.4)
- removed the JP2 at (99.3, 89.4)
- U1, U2, U3: footprint boardloaf-he-CustomFoot:SOIC-16_3.9x9.9mm_P1.27mm -> boardloaf-he-CustomFoot:reversible-SOIC-16_3.9x9.9mm_P1.27mm
- moved C19 46.9 mm to (70.2, 28.2), turned to 90 degrees
- moved U1 40.9 mm to (70.3, 35.4), turned to 0 degrees
- moved C20 26.3 mm to (70.3, 47.3), turned to 90 degrees
- moved U2 24.5 mm to (70.3, 54.4), turned to 0 degrees
- moved U3 17.4 mm to (70.2, 73.8), turned to 0 degrees
- moved C21 13.4 mm to (70.2, 66.7), turned to 90 degrees
- renumbered JP3 to JP1, JP4 to JP2
Connections:
- J1 pad S: Net-(JP2-A) -> GND
- J1 pad T: Net-(JP1-A) -> GND
- J2 pad S: Net-(JP1-A) -> GND
- J2 pad T: Net-(JP2-A) -> GND
Routing:
- net VCC: track 0.00 -> 484.4 mm, vias 5 -> 6
- net SEL0: track 0.00 -> 115.1 mm, vias 2 -> 3
- net SEL1: track 0.00 -> 100.9 mm, vias 4 -> 3
- net VAL0: track 0.00 -> 96.1 mm
- net SEL2: track 0.00 -> 94.9 mm, vias 4 -> 3
- net Net-(SW16-VOUT): track 0.00 -> 88.3 mm, vias 2 -> 4
- net VAL1: track 0.00 -> 80.3 mm
- net SERIAL: track 0.00 -> 61.9 mm
- net Net-(SW17-VOUT): track 0.00 -> 55.6 mm, vias 2 -> 1
- net VAL2: track 0.00 -> 55.2 mm
- net Net-(SW6-VOUT): track 0.00 -> 54.2 mm, vias 2 -> 0
- net Net-(SW18-VOUT): track 0.00 -> 54.0 mm
- net Net-(SW1-VOUT): track 0.00 -> 53.9 mm, vias 2 -> 0
- net Net-(SW11-VOUT): track 0.00 -> 53.6 mm, vias 2 -> 0
- net GND: track 0.00 -> 37.1 mm, vias 31 -> 30
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Other:
- board text added: "Rev 1.1"

Commit message: Rev 2 hardware draft
Connections:
- J1 pad R1: SERIAL -> GND
- J1 pad S: GND -> TX
- J1 pad T: GND -> RX
- J2 pad R1: SERIAL -> GND
- J2 pad S: GND -> RX
- J2 pad T: GND -> TX
- MCU1 pad 0: unconnected-(MCU1-Pad0) -> TX
- MCU1 pad 1: unconnected-(MCU1-Pad1) -> RX
- MCU1 pad 14: SERIAL -> unconnected-(MCU1-Pad14)
Routing:
- net TX: track 0.00 -> 63.8 mm, vias 0 -> 1
- net SERIAL: track 61.9 -> 0.00 mm
- net RX: track 0.00 -> 60.3 mm, vias 0 -> 1
- net Net-(SW18-VOUT): track 54.0 -> 57.6 mm, vias 0 -> 2
Other:
- board text added: "Rev 2.0"
- board text removed: "Rev 1.1"
