File: kicad/boardloaf-he.kicad_sch (KiCad schematic)
At the start: 49 parts, among them J1 AudioJack4, J2 AudioJack4, SW1 SLSS49E, SW10 SLSS49E, SW11 SLSS49E, SW12 SLSS49E, SW13 SLSS49E, SW14 SLSS49E, SW15 SLSS49E, SW16 SLSS49E, SW17 SLSS49E, SW18 SLSS49E, SW2 SLSS49E, SW3 SLSS49E, SW4 SLSS49E, SW5 SLSS49E, SW6 SLSS49E, SW7 SLSS49E, SW8 SLSS49E, SW9 SLSS49E, U1 74HC4051, U2 74HC4051, U3 74HC4051

Commit message: Made schematic sync with PCB
Parts:
- C1, C10, C11, C12, C13, C14, C15, C16, C17, C18, C19, C2, C20, C21, C3, C4, C5, C6, C7, C8, C9: footprint Capacitor_SMD:C_0805_2012Metric_Pad1.18x1.45mm_HandSolder -> boardloaf-he-CustomFoot:C_0805_2012Metric_Pad1.18x1.45mm_HandSolder
- J1, J2: footprint (none) -> boardloaf-he-CustomFoot:TRRS-PJ-320A_PIN
- JP1, JP2, JP3, JP4: footprint (none) -> Jumper:SolderJumper-2_P1.3mm_Open_TrianglePad1.0x1.5mm
- MCU1: renamed from MCU; footprint (none) -> boardloaf-he-CustomFoot:RP2040-Zero-RESIZED
- SW1, SW10, SW11, SW12, SW13, SW14, SW15, SW16, SW17, SW18, SW2, SW3, SW4, SW5, SW6, SW7, SW8, SW9: footprint project-specific-library:HE-Switch-1U -> boardloaf-he-CustomFoot:HE-Switch-1U
- U1, U2, U3: footprint Package_SO:SOIC-16_3.9x9.9mm_P1.27mm -> boardloaf-he-CustomFoot:SOIC-16_3.9x9.9mm_P1.27mm

Commit message: Rev 1.1 draft. Mux on both sides
Parts:
- removed JP1, JP2: SolderJumper_2_Open, Jumper:SolderJumper-2_P1.3mm_Open_TrianglePad1.0x1.5mm, symbol Jumper:SolderJumper_2_Open
- U1, U2, U3: footprint boardloaf-he-CustomFoot:SOIC-16_3.9x9.9mm_P1.27mm -> boardloaf-he-CustomFoot:reversible-SOIC-16_3.9x9.9mm_P1.27mm
- renumbered JP3 to JP1, JP4 to JP2
Connections:
- net GND: now also J1.S, J1.T, J2.S, J2.T

Commit message: Rev 2 hardware draft
Connections:
- net GND: now also J1.R1, J2.R1; no longer J1.S, J1.T, J2.S, J2.T
- net TX: now reaches MCU1.0
- net TX: now also J1.S, J2.T
- net RX: now reaches MCU1.1
- net RX: now also J1.T, J2.S
- removed net SERIAL: J1.R1, J2.R1, MCU1.14
- no-connect marks 13 -> 12
